File: type-c-battery.sch (KiCad schematic (older format))
At the start: 16 parts, among them J1 BAT, J2 USB Type-C Receptacle, U1 AP2161, U2 TP4055, U3 TUSB320HA

Commit message: boost design
Parts:
- removed R1: 200k, kicad-libs:SMD-1005, symbol Rs
- removed U1: AP2161, kicad-libs:SOT-23-5, symbol AP2161
- added C6: 22p, kicad-libs:SMD-1005, symbol C
- added C7: 10u, kicad-libs:SMD-2012, symbol C
- added L1: 2.2u, kicad-libs:SMD-3225, symbol L
- added Q1, Q2: DMP2035U, kicad-libs:SOT-23-FET, symbol PMOS
- added R1: 750k, kicad-libs:SMD-1005, symbol R
- added R2: 100k, kicad-libs:SMD-1005, symbol R
- added R7, R9: 900k, kicad-libs:SMD-1005, symbol R
- added R8: 66k, kicad-libs:SMD-1005, symbol R
- added U1: PAM2401-DFN, symbol PAM2401-DFN
- added U4: 74AHC1G04, kicad-libs:SC-70-5, symbol 74xx1G04
- C1: value 0.1u -> 22u; footprint kicad-libs:SMD-1005 -> kicad-libs:SMD-3216; Manufacturer (none) -> Samsung; Part Number (none) -> CL31X226KQHNNNE
- C2: Manufacturer (none) -> AVX; Part Number (none) -> TCJB157M006R0055
- C3, C4: value 10u -> 4.7u; Manufacturer (none) -> Samsung; Part Number (none) -> CL10B475KQ8NQNC
- J1: Manufacturer (none) -> JST; Part Number (none) -> S2B-PH-SM4-TB(LF)(SN)
- J2: Manufacturer (none) -> JAE; Part Number (none) -> DX07B024JJ2R1500
- R4, R5: symbol Rs -> R
- U3: Manufacturer (none) -> TI; Part Number (none) -> TUSB320HAIRWBR
- renumbered R2 to R6
Connections:
- net COM: now also C7.2, R2.2, R8.2, U1.11 (PGND), U1.12 (PGND), U1.6 (AGND), U1.FLAG (GND), U4.3
- net VBAT: now also C7.1, L1.2, R9.1, U1.4 (VIN), U4.5; no longer C1.1, C2.+
- net VBUS: now also Q1.S, Q2.S, R7.1; no longer C3.1, R6.1, U2.4 (VCC)
- net ~DFP: now also R9.2, U4.2
- new net: C3.1, Q2.D, R6.1, U2.4 (VCC)
- new net: C1.1, C2.+, C6.1, Q1.D, Q2.G, R1.1, U1.10 (OUT), U1.9 (OUT)
- new net: L1.1, U1.1 (LX), U1.2 (LX)
- new net: C6.2, R1.2, R2.1, U1.7 (FB)
- new net: R8.1, U1.8 (RSET)
- new net DFP: U1.3 (EN), U4.4
- new net ~PG: Q1.G, R7.2, U1.5 (PG)
Other:
- note added: "66k = 1A"
- moved on the sheet: C1, C2, C3, C4, D1, J1, J2, R3, R4, R5, R6, U2
