File: type-c-battery.sch (KiCad schematic (older format))
At the start: 26 parts, among them J1 BAT, J2 USB Type-C Receptacle, Q1 DMP2035U, Q2 DMP2035U, U1 PAM2401-DFN, U2 TP4055, U3 TUSB320HA, U4 74AHC1G04

Commit message: layout
Parts:
- removed R5: 200k, kicad-libs:SMD-1005, symbol R
- U1: footprint (none) -> kicad-libs:U-DFN3030-12
Connections:
- net VOUT: now reaches C1.1, C2.+, C6.1, Q1.D, Q2.G, R1.1, U1.10 (OUT), U1.9 (OUT)
- net LX: now reaches L1.1, U1.1 (LX), U1.2 (LX)
- net ~ERR: no longer names the net of U3.11 (EN)
- no-connect marks 19 -> 20
Changed lines of the file:
@@
 Sheet 1 1
 Title "USB Type-C LiPo DRP (boost)"
-Date "2017-07-03"
-Rev "r1"
+Date "2017-07-10"
+Rev "A0"
 Comp "sternlabs"
 Comment1 ""
@@
 Text Label 6550 4500 2    50   ~ 0
 ~DFP
-Text Label 4100 4900 0    50   ~ 0
-~ERR
-$Comp
-L R R5
-U 1 1 594EA592
-P 4450 4600
-F 0 "R5" H 4518 4496 50  0000 L CNN
-F 1 "200k" H 4518 4405 50  0000 L CNN
-F 2 "kicad-libs:SMD-1005" H 4585 4440 60  0001 C CNN
-F 3 "" H 4585 4440 60  0000 C CNN
-	1    4450 4600
-	1    0    0    -1
-$EndComp
-$Comp
-L VBAT #PWR016
-U 1 1 594EA756
-P 4450 4600
-F 0 "#PWR016" H 4460 4600 20  0001 C CNN
-F 1 "VBAT" H 4450 4660 40  0000 C CNN
-F 2 "" H 4450 4600 60  0000 C CNN
-F 3 "" H 4450 4600 60  0000 C CNN
-	1    4450 4600
-	1    0    0    -1
-$EndComp
 NoConn ~ 5950 4600
 NoConn ~ 5950 4700
 NoConn ~ 5950 4800
 $Comp
-L VBUS #PWR017
+L VBUS #PWR016
 U 1 1 594EAAC8
 P 4800 4000
-F 0 "#PWR017" H 4810 4000 20  0001 C CNN
+F 0 "#PWR016" H 4810 4000 20  0001 C CNN
 F 1 "VBUS" H 4800 4060 40  0000 C CNN
 F 2 "" H 4800 4000 60  0000 C CNN
@@
 $EndComp
 $Comp
-L COM #PWR018
+L COM #PWR017
 U 1 1 594EAC74
 P 5600 1600
-F 0 "#PWR018" V 5875 1600 60  0001 C CNN
+F 0 "#PWR017" V 5875 1600 60  0001 C CNN
 F 1 "COM" H 5760 1485 30  0001 C CNN
 F 2 "" H 5755 1610 60  0000 C CNN
@@
 $EndComp
 $Comp
-L COM #PWR019
+L COM #PWR018
 U 1 1 594EADB2
 P 6900 3200
-F 0 "#PWR019" V 7175 3200 60  0001 C CNN
+F 0 "#PWR018" V 7175 3200 60  0001 C CNN
 F 1 "COM" H 7060 3085 30  0001 C CNN
 F 2 "" H 7055 3210 60  0000 C CNN
@@
 $EndComp
 $Comp
-L COM #PWR020
+L COM #PWR019
 U 1 1 594EB837
 P 6100 4400
-F 0 "#PWR020" V 6375 4400 60  0001 C CNN
+F 0 "#PWR019" V 6375 4400 60  0001 C CNN
 F 1 "COM" H 6260 4285 30  0001 C CNN
 F 2 "" H 6255 4410 60  0000 C CNN
@@
 $EndComp
 $Comp
-L COM #PWR021
+L COM #PWR020
 U 1 1 594EBBFB
 P 5950 1600
-F 0 "#PWR021" V 6225 1600 60  0001 C CNN
+F 0 "#PWR020" V 6225 1600 60  0001 C CNN
 F 1 "COM" H 6110 1485 30  0001 C CNN
 F 2 "" H 6105 1610 60  0000 C CNN
@@
 $EndComp
 $Comp
-L POWER_FLAG #PWR022
+L POWER_FLAG #PWR021
 U 1 1 594EBE5F
 P 10250 2300
-F 0 "#PWR022" H 10250 2300 50  0001 C CNN
+F 0 "#PWR021" H 10250 2300 50  0001 C CNN
 F 1 "POWER_FLAG" H 10245 2458 30  0000 C CNN
 F 2 "" H 10250 2300 50  0000 C CNN
@@
 $EndComp
 $Comp
-L COM #PWR023
+L COM #PWR022
 U 1 1 594EBE91
 P 10250 2300
-F 0 "#PWR023" V 10525 2300 60  0001 C CNN
+F 0 "#PWR022" V 10525 2300 60  0001 C CNN
 F 1 "COM" H 10410 2185 30  0001 C CNN
 F 2 "" H 10405 2310 60  0000 C CNN
@@
 $EndComp
 $Comp
-L COM #PWR024
+L COM #PWR023
 U 1 1 594EF924
 P 2600 3200
-F 0 "#PWR024" V 2875 3200 60  0001 C CNN
+F 0 "#PWR023" V 2875 3200 60  0001 C CNN
 F 1 "COM" H 2760 3085 30  0001 C CNN
 F 2 "" H 2755 3210 60  0000 C CNN
@@
 F 0 "U1" H 7350 2387 60  0000 C CNN
 F 1 "PAM2401-DFN" H 7350 2281 60  0000 C CNN
-F 2 "" H 7350 2250 60  0001 C CNN
+F 2 "kicad-libs:U-DFN3030-12" H 7350 2250 60  0001 C CNN
 F 3 "" H 7350 2250 60  0001 C CNN
 F 4 "PAM2401YPADJ" H 0   0   60  0001 C CNN "Part Number"
@@
 $EndComp
 $Comp
-L COM #PWR025
+L COM #PWR024
 U 1 1 595984A5
 P 6850 2150
-F 0 "#PWR025" V 7125 2150 60  0001 C CNN
+F 0 "#PWR024" V 7125 2150 60  0001 C CNN
 F 1 "COM" H 7010 2035 30  0001 C CNN
 F 2 "" H 7005 2160 60  0000 C CNN
@@
 $EndComp
 $Comp
-L COM #PWR026
+L COM #PWR025
 U 1 1 595985A3
 P 6500 2000
-F 0 "#PWR026" V 6775 2000 60  0001 C CNN
+F 0 "#PWR025" V 6775 2000 60  0001 C CNN
 F 1 "COM" H 6660 1885 30  0001 C CNN
 F 2 "" H 6655 2010 60  0000 C CNN
@@
 $EndComp
 $Comp
-L COM #PWR027
+L COM #PWR026
 U 1 1 59598F09
 P 8450 1600
-F 0 "#PWR027" V 8725 1600 60  0001 C CNN
+F 0 "#PWR026" V 8725 1600 60  0001 C CNN
 F 1 "COM" H 8610 1485 30  0001 C CNN
 F 2 "" H 8605 1610 60  0000 C CNN
@@
 $EndComp
 $Comp
-L COM #PWR028
+L COM #PWR027
 U 1 1 595990A9
 P 7900 2400
-F 0 "#PWR028" V 8175 2400 60  0001 C CNN
+F 0 "#PWR027" V 8175 2400 60  0001 C CNN
 F 1 "COM" H 8060 2285 30  0001 C CNN
 F 2 "" H 8055 2410 60  0000 C CNN
@@
 $EndComp
 $Comp
-L COM #PWR029
+L COM #PWR028
 U 1 1 5959BFBA
 P 7650 4650
-F 0 "#PWR029" V 7925 4650 60  0001 C CNN
+F 0 "#PWR028" V 7925 4650 60  0001 C CNN
 F 1 "COM" H 7810 4535 30  0001 C CNN
 F 2 "" H 7805 4660 60  0000 C CNN
@@
 $EndComp
 $Comp
-L VBAT #PWR030
+L VBAT #PWR029
 U 1 1 5959C5FD
 P 7650 4350
-F 0 "#PWR030" H 7660 4350 20  0001 C CNN
+F 0 "#PWR029" H 7660 4350 20  0001 C CNN
 F 1 "VBAT" H 7650 4410 40  0000 C CNN
 F 2 "" H 7650 4350 60  0000 C CNN
@@
 DFP
 $Comp
-L VBAT #PWR031
+L VBAT #PWR030
 U 1 1 5959CB2F
 P 7350 4200
-F 0 "#PWR031" H 7360 4200 20  0001 C CNN
+F 0 "#PWR030" H 7360 4200 20  0001 C CNN
 F 1 "VBAT" H 7350 4260 40  0000 C CNN
 F 2 "" H 7350 4200 60  0000 C CNN
@@
 ~PG
 $Comp
-L POWER_FLAG #PWR032
+L POWER_FLAG #PWR031
 U 1 1 5959FBF7
 P 3750 2200
-F 0 "#PWR032" H 3750 2200 50  0001 C CNN
+F 0 "#PWR031" H 3750 2200 50  0001 C CNN
 F 1 "POWER_FLAG" H 3745 2358 30  0000 C CNN
 F 2 "" H 3750 2200 50  0000 C CNN
@@
 $EndComp
 $Comp
-L POWER_FLAG #PWR033
+L POWER_FLAG #PWR032
 U 1 1 5959FF6E
 P 7200 3000
-F 0 "#PWR033" H 7200 3000 50  0001 C CNN
+F 0 "#PWR032" H 7200 3000 50  0001 C CNN
 F 1 "POWER_FLAG" H 7195 3158 30  0000 C CNN
 F 2 "" H 7200 3000 50  0000 C CNN
@@
 Wire Wire Line
 	6550 4500 5950 4500
-Wire Wire Line
-	4100 4900 4950 4900
-Connection ~ 4450 4900
 Connection ~ 5600 1400
 Connection ~ 6900 3000
@@
 Entry Wire Line
 	11800 7000 11900 7100
+NoConn ~ 4950 4900
+Text Label 7850 1400 0    50   ~ 0
+LX
+Text Label 6800 1400 2    50   ~ 0
+VOUT
 $EndSCHEMATC
