File: type-c-battery.sch (KiCad schematic (older format))
At the start: 16 parts, among them J1 BAT, J2 USB Type-C Receptacle, U1 AP2161, U2 TP4055, U3 TUSB320HA

Commit message: BOM
Parts:
- C2: Manufacturer (none) -> AVX; Part Number (none) -> TCJB157M006R0055
- C3, C4: value 10u -> 4.7u; Manufacturer (none) -> Samsung; Part Number (none) -> CL10B475KQ8NQNC
- J1: Manufacturer (none) -> JST; Part Number (none) -> S2B-PH-SM4-TB(LF)(SN)
- J2: Manufacturer (none) -> JAE; Part Number (none) -> DX07B024JJ2R1500
- U1: Manufacturer (none) -> Diodes; Part Number (none) -> AP2161WG-7
- U3: Manufacturer (none) -> TI; Part Number (none) -> TUSB320HAIRWBR
Changed lines of the file:
@@
 EESchema Schematic File Version 2
+LIBS:74xx1g04
+LIBS:pam2401
 LIBS:ap2161
 LIBS:tusb320la
@@
 F 2 "kicad-libs:X2QFN-12" H 5450 5200 60  0001 C CNN
 F 3 "" H 5450 5200 60  0001 C CNN
+F 4 "TUSB320HAIRWBR" H 0   0   60  0001 C CNN "Part Number"
+F 5 "TI" H 0   0   60  0001 C CNN "Manufacturer"
 	1    5450 4650
 	1    0    0    -1
@@
 F 2 "kicad-libs:USB-TYPE-C-DX07B024JJ1" H 2550 3350 50  0001 C CNN
 F 3 "" H 2550 3350 50  0001 C CNN
+F 4 "DX07B024JJ2R1500" H 0   0   60  0001 C CNN "Part Number"
+F 5 "JAE" H 0   0   60  0001 C CNN "Manufacturer"
 	1    2550 2650
 	1    0    0    -1
@@
 F 2 "kicad-libs:JST-PH-2-RIGHT-SMD" H 9600 2450 60  0001 C CNN
 F 3 "" H 9600 2450 60  0000 C CNN
+F 4 "S2B-PH-SM4-TB(LF)(SN)" H 0   0   60  0001 C CNN "Part Number"
+F 5 "JST" H 0   0   60  0001 C CNN "Manufacturer"
 	1    9600 2450
 	1    0    0    1
@@
 P 8600 2850
 F 0 "C4" H 8673 2796 50  0000 L CNN
-F 1 "10u" H 8673 2705 50  0000 L CNN
+F 1 "4.7u" H 8673 2705 50  0000 L CNN
 F 2 "kicad-libs:SMD-1608" H 8500 3000 60  0001 C CNN
 F 3 "" H 8500 3000 60  0000 C CNN
+F 4 "CL10B475KQ8NQNC" H 0   0   60  0001 C CNN "Part Number"
+F 5 "Samsung" H 0   0   60  0001 C CNN "Manufacturer"
 	1    8600 2850
 	1    0    0    -1
@@
 F 2 "kicad-libs:SOT-23-5" H 6450 2300 60  0001 C CNN
 F 3 "" H 6450 2300 60  0001 C CNN
+F 4 "AP2161WG-7" H 0   0   60  0001 C CNN "Part Number"
+F 5 "Diodes" H 0   0   60  0001 C CNN "Manufacturer"
 	1    6450 2050
 	-1   0    0    -1
@@
 F 2 "kicad-libs:SMD-3528-CP" H 7800 2100 60  0001 C CNN
 F 3 "" H 7800 2100 60  0000 C CNN
+F 4 "TCJB157M006R0055" H 0   0   60  0001 C CNN "Part Number"
+F 5 "AVX" H 0   0   60  0001 C CNN "Manufacturer"
 	1    7900 1950
 	1    0    0    -1
@@
 P 6900 2850
 F 0 "C3" H 6973 2796 50  0000 L CNN
-F 1 "10u" H 6973 2705 50  0000 L CNN
+F 1 "4.7u" H 6973 2705 50  0000 L CNN
 F 2 "kicad-libs:SMD-1608" H 6800 3000 60  0001 C CNN
 F 3 "" H 6800 3000 60  0000 C CNN
+F 4 "CL10B475KQ8NQNC" H 0   0   60  0001 C CNN "Part Number"
+F 5 "Samsung" H 0   0   60  0001 C CNN "Manufacturer"
 	1    6900 2850
 	1    0    0    -1
