File: type-c-battery.kicad_pcb (KiCad board)
At the start: 2 copper layers, 28 x 14 mm, 17 parts, among them J1 BAT, J2 USB Type-C Receptacle, U1 AP2161, U2 TP4055, U3 TUSB320HA

Commit message: layout
Parts:
- removed R5: 200k, kicad-libs:SMD-1005
- added C6: 22p, kicad-libs:SMD-1005, F.Cu at (149.8, 82.2)
- added C7: 10u, kicad-libs:SMD-2012, F.Cu at (154.5, 86.2)
- added L1: 2.2u, kicad-libs:SMD-3225, F.Cu at (158.0, 85.2)
- added Q1: DMP2035U, kicad-libs:SOT-23-FET, F.Cu at (147.5, 81.5)
- added Q2: DMP2035U, kicad-libs:SOT-23-FET, F.Cu at (151.2, 90.5)
- added R6: 5k, kicad-libs:SMD-1005, F.Cu at (162.2, 84.5)
- added R7: 900k, kicad-libs:SMD-1005, F.Cu at (150.2, 80.8)
- added R8: 66k, kicad-libs:SMD-1005, F.Cu at (153.2, 80.2)
- added R9: 900k, kicad-libs:SMD-1005, F.Cu at (160.2, 81.0)
- added U4: 74AHC1G04, kicad-libs:SC-70-5, F.Cu at (157.8, 81.0)
- C1: value 0.1u -> 22u; footprint kicad-libs:SMD-1005 -> kicad-libs:SMD-3216
- C3, C4: value 10u -> 4.7u
- R1: value 200k -> 750k
- R2: value 5k -> 100k
- U1: value AP2161 -> PAM2401-DFN; footprint kicad-libs:SOT-23-5 -> kicad-libs:U-DFN3030-12
- moved R2 9.74 mm to (153.2, 81.2)
- moved C2 6.27 mm to (147.5, 85.8), turned to 270 degrees
- moved U1 6.18 mm to (153.8, 83.5), turned to 90 degrees
- moved C4 6.05 mm to (153.0, 96.0), turned to 90 degrees
- moved R3 5.48 mm to (149.0, 91.2), turned to 180 degrees
- moved R1 5.15 mm to (150.8, 82.2), turned to 180 degrees
- moved U2 3.18 mm to (150.0, 94.5), turned to 0 degrees
- moved C3 2.25 mm to (152.2, 93.8), turned to 0 degrees
- moved G*** 2.06 mm to (155.2, 87.8)
- moved J2 1.75 mm to (138.2, 88.2)
- moved D1 1.58 mm to (162.2, 83.0), turned to 90 degrees
- moved C1 0.75 mm to (150.5, 85.8)
Connections:
- C1 pad 1: VBAT -> /VOUT
- C2 pad +: VBAT -> /VOUT
- C3 pad 1: VBUS -> Net-(C3-Pad1)
- R1 pad 1: VBAT -> /VOUT
- R1 pad 2: /~DFP -> Net-(C6-Pad2)
- R2 pad 1: VBUS -> Net-(C6-Pad2)
- R2 pad 2: Net-(D1-PadA) -> COM
- U1 pad 1: VBUS -> /LX
- U1 pad 2: COM -> /LX
- U1 pad 3: /~ERR -> /DFP
- U1 pad 4: /~DFP -> VBAT
- U1 pad 5: VBAT -> /~PG
- U2 pad 4: VBUS -> Net-(C3-Pad1)
- U3 pad 11: /~ERR -> Net-(U3-Pad11)
Routing:
- net /~DFP: track 9.21 -> 43.7 mm
- net Net-(C3-Pad1): track 0.00 -> 28.7 mm, vias 0 -> 2
- net /VOUT: track 0.00 -> 14.9 mm
- net /~PG: track 0.00 -> 12.9 mm, vias 0 -> 2
- net VBUS: track 43.4 -> 31.2 mm
- net Net-(D1-PadC): track 17.0 -> 29.0 mm, vias 0 -> 2
- net COM: track 23.0 -> 33.1 mm, vias 18 -> 27
- net /~ERR: track 9.15 -> 0.00 mm, vias 2 -> 0
- net VBAT: track 25.9 -> 34.5 mm
- net /DFP: track 0.00 -> 4.61 mm
- net Net-(C6-Pad2): track 0.00 -> 3.90 mm
- net Net-(R8-Pad1): track 0.00 -> 3.69 mm, vias 0 -> 2
- net /CC1: track 6.30 -> 8.05 mm
- net /CC2: track 5.99 -> 7.65 mm
- added copper zone on F.Cu, net /LX
- added copper zone on F.Cu, net /VOUT
Other:
- board size 28 x 14 mm -> 28 x 17.5 mm
- board text added: "Type-C LiPo DRP (boost) rev A0"
- board text removed: "Type-C LiPo DRP (non-boost) rev A0"
