File: type-c-battery.kicad_pcb (KiCad board)
At the start: 2 copper layers, 28 x 14 mm, 17 parts, among them J1 BAT, J2 USB Type-C Receptacle, U1 AP2161, U2 TP4055, U3 TUSB320HA

Commit message: update cap values
Parts:
- C3, C4: value 10u -> 4.7u
Changed lines of the file:
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@@
-(kicad_pcb (version 20170123) (host pcbnew "(2017-06-02 revision ac9a64a17)-master")
+(kicad_pcb (version 20170123) (host pcbnew "(2017-07-06 revision 885a4c1bc)-master")
   (general
-    (links 50)
-    (no_connects 0)
-    (area 136.099999 80.655952 166.675001 99.344047)
     (thickness 1.6)
     (drawings 5)
@@
   )
   (page A4)
+  (title_block
+    (title "USB Type-C LiPo DRP (non-boost)")
+    (date 2017-07-14)
+    (rev A0)
+  )
   (layers
     (0 F.Cu signal)
@@
     (add_net VBUS)
   )
-  (module kicad-libs:starfish2-10 (layer B.Cu)
+  (module kicad-libs:starfish2-10 locked (layer B.Cu)
     (at 155.75 89.75 270)
     (fp_text reference G*** (at 0 0 270) (layer B.SilkS) hide
@@
       (effects (font (size 0.7 0.7) (thickness 0.15)))
     )
-    (fp_text value 10u (at 0 0 90) (layer F.Fab) hide
+    (fp_text value 4.7u (at 0 0 90) (layer F.Fab) hide
       (effects (font (size 0.7 0.7) (thickness 0.15)))
     )
@@
       (effects (font (size 0.7 0.7) (thickness 0.15)))
     )
-    (fp_text value 10u (at 0 0 270) (layer F.Fab) hide
-      (effects (font (size 0.7 0.7) (thickness 0.15)))
-    )
+    (fp_text value 4.7u (at 0 0 270) (layer F.Fab) hide
+      (effects (font (size 0.7 0.7) (thickness 0.15)))
+    )
